File: Sensor_Board.kicad_pcb (KiCad board)
At the start: 4 copper layers, 100 x 100 mm, 252 parts, among them J1001 USB_B, J1101 VN_1611_Interface, J1102 AMPSEAL_35, J1103 Banana_Jack, J1104 Banana_Jack, Q1201 IPD50P04P413ATMA2, Q501 BTN8962TA, Q502 BTN8962TA, Q601 BC817, Q602 BC817, Q603 BC817, Q604 BC817, Q605 BC817, Q606 BC817, Q607 BC817, Q608 BC817, Q609 BC807, Q610 BC807, Q611 BC807, Q612 BC807, Q613 BC817, Q614 BC817, Q615 BC817, Q616 BC817, Q617 BC817, Q618 BC817, Q619 BC817, Q620 BC817, Q621 BC807, Q622 BC807, Q623 BC807, Q624 BC807, Q801 BSS123, Q802 BSS123, U1201 LM53603, U1202 LD1117S50TR_SOT223, U1203 LD1117S50TR_SOT223, U1204 LD1117S33TR_SOT223, U201 74HC595, U301 74HC595, U302 74HCT244, U401 TLE9351VSJ, U402 TLE7258SJ, U501 BTT6200-4ESA, U701 24LC32, U801 74LS125, U802 MAX11614, U901 STM32F103RBTx

Commit message: placed components and began routing
Parts:
- removed JP501: SolderJumper_3_Open, Jumper:SolderJumper-3_P1.3mm_Open_Pad1.0x1.5mm
- added C1001: 100nF, Capacitor_SMD:C_0603_1608Metric, F.Cu at (122.0, 122.0)
- added C1201: 470nF, Capacitor_SMD:C_0805_2012Metric, F.Cu at (57.0, 53.0)
- added C1203: 22µ, Capacitor_SMD:C_1210_3225Metric, F.Cu at (64.5, 46.5)
- added C1204: 22µ, Capacitor_SMD:C_1210_3225Metric, F.Cu at (72.0, 46.5)
- added C1205: 22µ, Capacitor_SMD:C_1210_3225Metric, F.Cu at (68.5, 46.5)
- added C1210: 3.3µF, Capacitor_SMD:C_1206_3216Metric, F.Cu at (53.0, 55.0)
- added C1213: 22µ, Capacitor_SMD:C_1210_3225Metric, B.Cu at (114.0, 130.8)
- added C1215: 22µ, Capacitor_SMD:C_1210_3225Metric, B.Cu at (114.0, 119.0)
- added C1217: 22µ, Capacitor_SMD:C_1210_3225Metric, B.Cu at (119.0, 105.0)
- added C501: 220µ, Capacitor_SMD:CP_Elec_10x10.5, F.Cu at (112.5, 71.9)
- added C507: 220µ, Capacitor_SMD:CP_Elec_10x10.5, F.Cu at (99.5, 71.9)
- added C508: 100nF, Capacitor_SMD:C_0603_1608Metric, B.Cu at (95.5, 55.4)
- added C509: 100nF, Capacitor_SMD:C_0603_1608Metric, B.Cu at (103.5, 55.4)
- added C510: 100nF, Capacitor_SMD:C_0603_1608Metric, F.Cu at (104.5, 62.9)
- added C511: 100nF, Capacitor_SMD:C_0603_1608Metric, B.Cu at (117.0, 55.4)
- added C512: 100nF, Capacitor_SMD:C_0603_1608Metric, B.Cu at (109.0, 55.4)
- added C513: 100nF, Capacitor_SMD:C_0603_1608Metric, F.Cu at (118.0, 62.9)
- added C514: 10n, Capacitor_SMD:C_0603_1608Metric, B.Cu at (91.5, 55.5)
- added C515: 10n, Capacitor_SMD:C_0603_1608Metric, B.Cu at (88.0, 55.5)
- added C516: 10n, Capacitor_SMD:C_0603_1608Metric, B.Cu at (84.5, 55.5)
- added C517: 10n, Capacitor_SMD:C_0603_1608Metric, B.Cu at (81.0, 54.0)
- added C518: 100nF, Capacitor_SMD:C_0603_1608Metric, F.Cu at (81.3, 60.0)
- added C519: 1µ, Capacitor_SMD:C_0603_1608Metric, F.Cu at (79.3, 60.0)
- added C901: 100nF, Capacitor_SMD:C_0603_1608Metric, F.Cu at (117.5, 96.0)
- added C902: 100nF, Capacitor_SMD:C_0603_1608Metric, F.Cu at (103.5, 111.0)
- added C903: 100nF, Capacitor_SMD:C_0603_1608Metric, F.Cu at (103.5, 91.0)
- added C904: 100nF, Capacitor_SMD:C_0603_1608Metric, F.Cu at (111.5, 111.0)
- added C906: 4.7µ, Capacitor_SMD:C_0603_1608Metric, F.Cu at (101.5, 91.0)
- added C907: 10n, Capacitor_SMD:C_0603_1608Metric, F.Cu at (97.5, 103.0)
- added C908: 1µ, Capacitor_SMD:C_0603_1608Metric, F.Cu at (97.5, 105.0)
- added C909: 100nF, Capacitor_SMD:C_0603_1608Metric, F.Cu at (97.5, 96.0)
- added C910: 100nF, Capacitor_SMD:C_0603_1608Metric, F.Cu at (93.5, 96.0)
- added C911: 100nF, Capacitor_SMD:C_0603_1608Metric, F.Cu at (93.5, 104.0)
- added D1206: GREEN, LED_SMD:LED_0603_1608Metric, F.Cu at (130.2, 154.3)
- added D1207: GREEN, LED_SMD:LED_0603_1608Metric, F.Cu at (132.2, 154.3)
- added D1208: GREEN, LED_SMD:LED_0603_1608Metric, F.Cu at (134.2, 154.3)
- added D1209: GREEN, LED_SMD:LED_0603_1608Metric, F.Cu at (136.2, 154.3)
- added D1210: GREEN, LED_SMD:LED_0603_1608Metric, F.Cu at (128.2, 154.3)
- added D502: PMEG4010CEH, Diode_SMD:D_SOD-123F, F.Cu at (91.5, 54.0)
- added D503: PMEG4010CEH, Diode_SMD:D_SOD-123F, F.Cu at (88.0, 54.0)
- added D504: PMEG4010CEH, Diode_SMD:D_SOD-123F, F.Cu at (84.5, 54.0)
- added D506: BLUE, LED_SMD:LED_0603_1608Metric, F.Cu at (83.0, 45.0)
- added D507: BLUE, LED_SMD:LED_0603_1608Metric, F.Cu at (86.5, 45.0)
- added D508: BLUE, LED_SMD:LED_0603_1608Metric, F.Cu at (81.0, 49.5)
- added D509: BLUE, LED_SMD:LED_0603_1608Metric, F.Cu at (84.5, 49.5)
- added D510: BLUE, LED_SMD:LED_0603_1608Metric, F.Cu at (88.0, 49.5)
- added D511: BLUE, LED_SMD:LED_0603_1608Metric, F.Cu at (91.5, 49.5)
- added D512: RED, LED_SMD:LED_0603_1608Metric, F.Cu at (117.5, 102.0)
- added D513: PMEG4010CEH, Diode_SMD:D_SOD-123F, F.Cu at (81.0, 54.0)
- added F1201: 2A, Fuse:Fuse_1206_3216Metric, F.Cu at (76.5, 59.0)
- added F1202: 0.5A, Fuse:Fuse_1206_3216Metric, F.Cu at (76.0, 65.0)
- added F1203: 0.5A, Fuse:Fuse_1206_3216Metric, F.Cu at (119.5, 116.0)
- added F1204: 0.5A, Fuse:Fuse_1206_3216Metric, B.Cu at (110.5, 130.8)
- added F1205: 0.5A, Fuse:Fuse_1206_3216Metric, B.Cu at (110.5, 119.0)
- added F1206: 0.5A, Fuse:Fuse_1206_3216Metric, B.Cu at (122.5, 105.0)
- added J901: SWD_Conn, Connector_PinHeader_2.54mm:PinHeader_1x06_P2.54mm_Vertical, F.Cu at (118.7, 80.0)
- added JP901: SolderJumper_2_Open, Jumper:SolderJumper-2_P1.3mm_Open_Pad1.0x1.5mm, F.Cu at (117.3, 84.0)
- added L1201: 2.2µH, Inductor_SMD:L_Bourns_SRP7028A_7.3x6.6mm, F.Cu at (58.5, 46.5)
- added R1202: 3, Resistor_SMD:R_0603_1608Metric, F.Cu at (53.0, 58.5)
- added R1209: 10k, Resistor_SMD:R_0603_1608Metric, F.Cu at (130.2, 150.8)
- added R1210: 1k, Resistor_SMD:R_0603_1608Metric, F.Cu at (132.2, 150.8)
- added R1211: 1k, Resistor_SMD:R_0603_1608Metric, F.Cu at (134.2, 150.8)
- added R1212: 1k, Resistor_SMD:R_0603_1608Metric, F.Cu at (136.2, 150.8)
- added R1213: 10k, Resistor_SMD:R_0603_1608Metric, F.Cu at (128.2, 150.8)
- added R510: 100k, Resistor_SMD:R_0603_1608Metric, B.Cu at (91.5, 54.0)
- added R511: 100k, Resistor_SMD:R_0603_1608Metric, B.Cu at (88.0, 54.0)
- added R512: 100k, Resistor_SMD:R_0603_1608Metric, B.Cu at (84.5, 54.0)
- added R513: 100k, Resistor_SMD:R_0603_1608Metric, B.Cu at (81.0, 55.5)
- added R514: 10k, Resistor_SMD:R_0603_1608Metric, F.Cu at (89.8, 72.5)
- added R515: 10k, Resistor_SMD:R_0603_1608Metric, F.Cu at (91.8, 69.0)
- added R516: 10k, Resistor_SMD:R_0603_1608Metric, F.Cu at (81.8, 69.0)
- added R517: 10k, Resistor_SMD:R_0603_1608Metric, F.Cu at (83.8, 69.0)
- added R518: 10k, Resistor_SMD:R_0603_1608Metric, F.Cu at (89.8, 69.0)
- added R519: 10k, Resistor_SMD:R_0603_1608Metric, F.Cu at (91.8, 72.5)
- added R520: 10k, Resistor_SMD:R_0603_1608Metric, F.Cu at (87.8, 69.0)
- added R521: 27, Resistor_SMD:R_0603_1608Metric, F.Cu at (83.8, 72.5)
- added R522: 10k, Resistor_SMD:R_0603_1608Metric, F.Cu at (88.5, 45.0)
- added R523: 10k, Resistor_SMD:R_0603_1608Metric, F.Cu at (81.0, 45.0)
- added R524: 10k, Resistor_SMD:R_0603_1608Metric, B.Cu at (81.0, 52.5)
- added R525: 10k, Resistor_SMD:R_0603_1608Metric, B.Cu at (84.5, 52.5)
- added R526: 10k, Resistor_SMD:R_0603_1608Metric, B.Cu at (88.0, 52.5)
- added R527: 10k, Resistor_SMD:R_0603_1608Metric, B.Cu at (91.5, 52.5)
- added R528: 1k, Resistor_SMD:R_0603_1608Metric, F.Cu at (121.0, 102.0)
- added R901: t.b.d., Resistor_SMD:R_0603_1608Metric, F.Cu at (97.5, 101.0)
- added RN301: 10k, Resistor_SMD:R_Array_Convex_8x0602, F.Cu at (66.4, 140.6)
- added U1001: USBLC6-2P6, Package_TO_SOT_SMD:SOT-666, F.Cu at (122.0, 124.0)
- added Y901: 8MHz, Crystal:Crystal_SMD_3225-4Pin_3.2x2.5mm, F.Cu at (93.5, 100.0)
- C1212, C1214, C1216, C503, C505, C804, D1204, D1205, D601, D602, D603, D604, D605, D606, D607, D608, JP1202, Q601, Q602, Q603, Q604, Q605, Q606, Q607, Q608, Q609, Q610, Q611, Q612, Q613, Q614, Q615, Q616, Q617, Q618, Q619, Q620, Q621, Q622, Q623, Q624, R501, R502, R503, R504, R505, R506, R507, R508, R601, R602, R603, R604, R605, R606, R607, R608, R609, R610, R611, R612, R613, R614, R615, R616, R617, R618, R619, R620, R621, R622, R623, R624, R625, R626, R627, R628, R629, R630, R631, R632, R633, R634, R635, R636, R637, R638, R639, R640, R641, R642, R643, R644, R645, R646, R647, R648, R802, R803, R804, R805, U1202, U1203, U1204: moved to B.Cu
- C201, C802, U201: moved to F.Cu
- C502, C504: value 100nF -> 1n; moved to B.Cu
- C506: value 100nF -> 100p
- D401: value D_TVS_Dual_AAC -> PESD2CANFD24V-T
- D402, D501: value BAT60A -> PMEG4010CEH; footprint Diode_SMD:D_SOD-323 -> Diode_SMD:D_SOD-123F
- FL401: value Filter_EMI_LL_1423 -> WE 744222
- R509: value 1k -> 1.2k
- U302: footprint Package_SO:SOIC-16_3.9x9.9mm_P1.27mm -> Package_SO:SOIC-20W_7.5x12.8mm_P1.27mm
- moved C401 193.8 mm to (57.8, 87.0), turned to 180 degrees
- moved D402 190.6 mm to (61.5, 80.5)
- moved D310 188.8 mm to (67.5, 120.0), turned to 180 degrees
- moved D307 187.6 mm to (63.0, 120.0)
- moved R403 187.0 mm to (65.5, 86.0)
- moved R402 186.5 mm to (65.5, 88.0), turned to 180 degrees
- moved D306 182.8 mm to (67.5, 113.0), turned to 180 degrees
- moved D305 182.4 mm to (67.5, 106.0), turned to 180 degrees
- moved D314 182.3 mm to (79.0, 120.0)
- moved D313 181.9 mm to (79.0, 113.0)
- moved D303 181.8 mm to (63.0, 113.0)
- moved D302 181.4 mm to (63.0, 106.0)
- moved D301 181.2 mm to (63.0, 99.2)
- moved R404 179.9 mm to (73.5, 83.0), turned to 180 degrees
- moved R401 178.1 mm to (73.5, 91.0), turned to 180 degrees
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Connections:
- C307 pad 1: +3V3 -> +3.3V
- C308 pad 1: +3V3 -> +3.3V
- C402 pad 1: +3V3 -> +3.3V
- C701 pad 1: +3V3 -> +3.3V
- D304 pad 2: +3V3 -> +3.3V
- D305 pad 2: +3V3 -> +3.3V
- D306 pad 2: +3V3 -> +3.3V
- D310 pad 2: +3V3 -> +3.3V
- D311 pad 2: +3V3 -> +3.3V
- D312 pad 2: +3V3 -> +3.3V
- D315 pad 2: +3V3 -> +3.3V
- D316 pad 2: +3V3 -> +3.3V
- D501 pad 1: unconnected-(D501-K-Pad1) -> GND
- D501 pad 2: unconnected-(D501-A-Pad2) -> Net-(D501-A)
- FL401 pad 1: Net-(U401-CANL) -> Net-(U401-CANH)
- FL401 pad 2: Net-(U401-CANH) -> Net-(U401-CANL)
- FL401 pad 3: CAN_H -> CAN_L
- FL401 pad 4: CAN_L -> CAN_H
- J1102 pad 10: /Analog Inputs/A_In_02 -> /Analog Inputs/A_In_03
- J1102 pad 11: /Analog Inputs/A_In_05 -> /Analog Inputs/A_In_02
- J1102 pad 12: /Analog Inputs/A_In_06 -> +5VA
- J1102 pad 13: /Connectors/VIN -> Half1_OUT
- J1102 pad 14: 1A_Out0 -> GND
- J1102 pad 15: 1A_Out1 -> GND
- J1102 pad 16: LIN -> Vdrive
- J1102 pad 17: CAN_L -> /Connectors/D_IO_0
- J1102 pad 19: /Connectors/D_IO_6 -> /Connectors/D_IO_2
- J1102 pad 2: Half0_OUT -> /Connectors/VIN
- J1102 pad 20: Vdrive -> /Connectors/D_IO_3
- J1102 pad 21: /Analog Inputs/A_In_00 -> /Analog Inputs/A_In_01
- J1102 pad 22: /Analog Inputs/A_In_03 -> /Analog Inputs/A_In_00
- J1102 pad 23: /Analog Inputs/A_In_07 -> /Analog Inputs/A_In_04
- J1102 pad 24: GND -> Half0_OUT
- J1102 pad 26: 1A_Out2 -> GND
- J1102 pad 27: 1A_Out3 -> 1A_Out0
- J1102 pad 28: GND -> 1A_Out1
- J1102 pad 29: /Connectors/D_IO_2 -> 1A_Out2
- J1102 pad 3: Half1_OUT -> LIN
- J1102 pad 30: /Connectors/D_IO_3 -> 1A_Out3
- J1102 pad 31: /Connectors/D_IO_7 -> GND
- J1102 pad 33: /Analog Inputs/A_In_01 -> /Analog Inputs/A_In_05
- J1102 pad 34: /Analog Inputs/A_In_04 -> /Analog Inputs/A_In_06
- J1102 pad 35: +5VA -> /Analog Inputs/A_In_07
- J1102 pad 4: GND -> CAN_L
- J1102 pad 6: /Connectors/D_IO_0 -> /Connectors/D_IO_4
- J1102 pad 7: /Connectors/D_IO_4 -> /Connectors/D_IO_5
- J1102 pad 8: /Connectors/D_IO_5 -> /Connectors/D_IO_6
- J1102 pad 9: GND -> /Connectors/D_IO_7
- Q801 pad 1: +3V3 -> +3.3V
- Q802 pad 1: +3V3 -> +3.3V
- R1001 pad 2: Net-(J1001-D+) -> Net-(R1001-Pad2)
- R1002 pad 2: Net-(J1001-D-) -> Net-(R1002-Pad2)
- R405 pad 1: +3V3 -> +3.3V
- R509 pad 2: /Microcontroller/1A_IS -> Net-(U501-IS)
- R701 pad 1: +3V3 -> +3.3V
- R702 pad 1: +3V3 -> +3.3V
- R803 pad 1: +3V3 -> +3.3V
- R805 pad 1: +3V3 -> +3.3V
- U301 pad 10: +3V3 -> +3.3V
- U301 pad 16: +3V3 -> +3.3V
- U401 pad 5: +3V3 -> +3.3V
- U501 pad 10: /Microcontroller/1A_IN3 -> Net-(U501-IN3)
- U501 pad 11: /Microcontroller/1A_DSEL1 -> Net-(U501-DSEL1)
- U501 pad 2: /Microcontroller/1A_IN0 -> Net-(U501-IN0)
- U501 pad 4: GND -> Net-(U501-GND)
- U501 pad 5: /Microcontroller/1A_IN1 -> Net-(U501-IN1)
- U501 pad 6: Net-(JP501-C) -> +3.3V
- U501 pad 7: /Microcontroller/1A_IS -> Net-(U501-IS)
- U501 pad 8: /Microcontroller/1A_DSEL0 -> Net-(U501-DSEL0)
- U501 pad 9: /Microcontroller/1A_IN2 -> Net-(U501-IN2)
- U701 pad 3: +3V3 -> +3.3V
- U701 pad 8: +3V3 -> +3.3V
- U901 pad 28: /Microcontroller/EEPROM_SCL -> /EEPROM/EEPROM_WP
- U901 pad 29: /Microcontroller/EEPROM_SCL -> /EEPROM/EEPROM_SCL
- U901 pad 30: /Microcontroller/EEPROM_SCL -> /EEPROM/EEPROM_SDA
- U901 pad 46: unconnected-(U901-PA13-Pad46) -> /Microcontroller/SWDIO
- U901 pad 49: unconnected-(U901-PA14-Pad49) -> /Microcontroller/SWCLK
- U901 pad 5: unconnected-(U901-PD0-Pad5) -> Net-(U901-PD0)
- U901 pad 6: unconnected-(U901-PD1-Pad6) -> Net-(U901-PD1)
- U901 pad 7: unconnected-(U901-NRST-Pad7) -> /Microcontroller/NRST
Routing:
- net /Analog Inputs/A_In_07: track 0.00 -> 55.1 mm
- net /ADC/A_In_filt_05: track 0.00 -> 48.1 mm
- net /Digital Inputs/D_In_0_filt: track 0.00 -> 47.8 mm
- net /Connectors/D_IO_7: track 0.00 -> 47.8 mm
- net /Analog Inputs/A_In_06: track 0.00 -> 47.8 mm
- net /Analog Inputs/A_In_04: track 0.00 -> 45.9 mm
- net /Digital Inputs/D_In_4_filt: track 0.00 -> 43.5 mm
- net /Digital Inputs/D_In_1_filt: track 0.00 -> 43.3 mm
- net /Analog Inputs/A_In_00: track 0.00 -> 39.7 mm
- net /Connectors/D_IO_6: track 0.00 -> 39.1 mm
- net /Digital Inputs/D_In_2_filt: track 0.00 -> 38.6 mm
- net /Analog Inputs/A_In_05: track 0.00 -> 38.2 mm
- net /ADC/A_In_filt_06: track 0.00 -> 38.0 mm
- net /Digital Inputs/D_In_5_filt: track 0.00 -> 37.9 mm
- net /Connectors/D_IO_5: track 0.00 -> 34.4 mm
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- added copper zone on In2.Cu, net +3.3V
- added copper zone on In2.Cu, net +5VA
- added copper zone on F.Cu, net +BATT
- added copper zone on F.Cu, net /Connectors/VIN
- added copper zone on In2.Cu, net /Connectors/VIN
- added copper zone on In2.Cu, net /Digital Outputs/DOut_Supply0
- added copper zone on In2.Cu, net /Digital Outputs/DOut_Supply1
- added copper zone on F.Cu, net /Power Supply/6V_Buck
- added copper zone on F.Cu, net GND
- added copper zone on In1.Cu, net GND
- added copper zone on B.Cu, net Half0_OUT
- added copper zone on F.Cu, net Half0_OUT
- added copper zone on B.Cu, net Half1_OUT
- added copper zone on F.Cu, net Half1_OUT
- added copper zone on F.Cu, net Net-(C1201-Pad2)
- added copper zone on F.Cu, net VIN
- added copper zone on F.Cu, net Vdrive
